File: hardware/placas_individuales/DownConverter/imac_g3_down_converter_board_adapter_es.kicad_pcb (KiCad board)
At the start: 2 copper layers, 88 x 39 mm, 8 parts, among them J1 Screw_Terminal_01x10, J2 Screw_Terminal_01x04, J7 Conn_02x12_Top_Bottom, M1 Fan_Tacho_PWM

Commit message: Placas individuales: DRC revisado, .kicad_pro y Gerber en español listo para fabricar
- .kicad_pcb actualizados (J20 sin segmento de longitud 0, J7 pad 16 sólido en Down Converter, ajustes de máscara)
- Nuevo .kicad_pro por placa (cobre-borde 0,2 mm, alivios térmicos como aviso)
- fabricacion/*_gerber.zip: Gerbers + taladros PTH/NPTH desde el .kicad_pcb vigente; reemplazan los zips antiguos (los originales siguen en originales/)
- iBOM en español regenerado
- README y LEEME actualizados

Co-Authored-By: Claude Sonnet 5.5 <noreply@anthropic.com>
Claude-Session: https://claude.ai/code/session_01CUq9b9AsuT1a2cpCUYrCH3
Other:
- rule pad_to_mask_clearance: 0.051 -> 0
Changed lines of the file:
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@@
 		(rev "1")
 		(company "JJaroll.dev")
-		(comment 4 "JJaroll.dev")
 		(comment 1 "Original: qbancoffee/imac_g3_ivad_board_init (LGPL-3.0)")
 		(comment 2 "Traduccion al espanol y firma: JJaroll.dev")
+		(comment 4 "JJaroll.dev")
 	)
 	(layers
@@
 	)
 	(setup
-		(pad_to_mask_clearance 0.051)
-		(solder_mask_min_width 0.25)
-		(allow_soldermask_bridges_in_footprints no)
+		(pad_to_mask_clearance 0)
+		(allow_soldermask_bridges_in_footprints yes)
 		(tenting
 			(front yes)
@@
 			(disableapertmacros no)
 			(usegerberextensions no)
-			(usegerberattributes no)
+			(usegerberattributes yes)
 			(usegerberadvancedattributes no)
 			(creategerberjobfile no)
@@
 			(remove_unused_layers no)
 			(net "/GND")
+			(zone_connect 2)
 		)
 		(pad "17" thru_hole circle

Commit message: Placas individuales: expansión de máscara 0,051 mm (como el diseño original)
- pad_to_mask_clearance 0,051 en los tres .kicad_pcb
- Gerbers de máscara ajustados con utilidades/expandir_mascara.py y verificados contra los Gerbers originales (diferencia de área de ~19 mm² a ~1,7 mm² por capa)
- LEEME de fabricacion y utilidades actualizados

Co-Authored-By: Claude Sonnet 5.5 <noreply@anthropic.com>
Claude-Session: https://claude.ai/code/session_01CUq9b9AsuT1a2cpCUYrCH3
Other:
- rule pad_to_mask_clearance: 0 -> 0.051
Changed lines of the file:
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@@
 	)
 	(setup
-		(pad_to_mask_clearance 0)
+		(pad_to_mask_clearance 0.051)
 		(allow_soldermask_bridges_in_footprints yes)
 		(tenting
