File: hardware/placas_individuales/J20_video/imac_g3_333mhz_slot_loading_J20_adapter_board_es.kicad_pcb (KiCad board)
At the start: 2 copper layers, 82.5 x 52.5 mm, 22 parts, among them J1 Screw_Terminal_01x06, J2 Conn_02x10_Odd_Even, J3 Conn_02x03_Odd_Even, J4 DB15_Female_HighDensity, J5 Conn_02x03_Odd_Even, U1 ATmega328-PU, U2 LCC110, Y1 Crystal

Commit message: Placas individuales: DRC revisado, .kicad_pro y Gerber en español listo para fabricar
- .kicad_pcb actualizados (J20 sin segmento de longitud 0, J7 pad 16 sólido en Down Converter, ajustes de máscara)
- Nuevo .kicad_pro por placa (cobre-borde 0,2 mm, alivios térmicos como aviso)
- fabricacion/*_gerber.zip: Gerbers + taladros PTH/NPTH desde el .kicad_pcb vigente; reemplazan los zips antiguos (los originales siguen en originales/)
- iBOM en español regenerado
- README y LEEME actualizados

Co-Authored-By: Claude Sonnet 5.5 <noreply@anthropic.com>
Claude-Session: https://claude.ai/code/session_01CUq9b9AsuT1a2cpCUYrCH3
Other:
- rule pad_to_mask_clearance: 0.051 -> 0
Changed lines of the file:
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@@
 		(rev "3")
 		(company "JJaroll.dev")
-		(comment 3 "inicializa la placa IVAD y envia el EDID cuando se solicita.")
-		(comment 4 "Alimenta el ATmega328P desde el conector J20 y desde el conector VGA.")
 		(comment 1 "Original: qbancoffee/imac_g3_ivad_board_init (LGPL-3.0)")
 		(comment 2 "Traduccion al espanol y firma: JJaroll.dev")
+		(comment 3 "inicializa la placa IVAD y envia el EDID cuando se solicita.")
+		(comment 4 "Alimenta el ATmega328P desde el conector J20 y desde el conector VGA.")
 	)
 	(layers
@@
 	)
 	(setup
-		(pad_to_mask_clearance 0.051)
-		(solder_mask_min_width 0.25)
-		(allow_soldermask_bridges_in_footprints no)
+		(pad_to_mask_clearance 0)
+		(allow_soldermask_bridges_in_footprints yes)
 		(tenting
 			(front yes)
@@
 			(drillshape 0)
 			(scaleselection 1)
-			(outputdirectory "gerbers_enviar/")
+			(outputdirectory "gerbers/")
 		)
 	)
@@
 		(net "/GREEN")
 	)
-	(segment
-		(start 173.403 74.1538)
-		(end 173.403 74.1538)
-		(width 0.25)
-		(layer "B.Cu")
-		(net "/GREEN")
-	)

Commit message: Placas individuales: expansión de máscara 0,051 mm (como el diseño original)
- pad_to_mask_clearance 0,051 en los tres .kicad_pcb
- Gerbers de máscara ajustados con utilidades/expandir_mascara.py y verificados contra los Gerbers originales (diferencia de área de ~19 mm² a ~1,7 mm² por capa)
- LEEME de fabricacion y utilidades actualizados

Co-Authored-By: Claude Sonnet 5.5 <noreply@anthropic.com>
Claude-Session: https://claude.ai/code/session_01CUq9b9AsuT1a2cpCUYrCH3
Other:
- rule pad_to_mask_clearance: 0 -> 0.051
Changed lines of the file:
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@@
 	)
 	(setup
-		(pad_to_mask_clearance 0)
+		(pad_to_mask_clearance 0.051)
 		(allow_soldermask_bridges_in_footprints yes)
 		(tenting
