File: hardware/placas_individuales/J22_frontal_audio/imac_g3_slot_loading_J22_adapter_board_es.kicad_pcb (KiCad board)
At the start: 2 copper layers, 65 x 30 mm, 12 parts, among them J1 Conn_02x13_Odd_Even, J2 Screw_Terminal_01x10, J3 AudioJack3, J4 Conn_02x03_Odd_Even

Commit message: Placas individuales: DRC revisado, .kicad_pro y Gerber en español listo para fabricar
- .kicad_pcb actualizados (J20 sin segmento de longitud 0, J7 pad 16 sólido en Down Converter, ajustes de máscara)
- Nuevo .kicad_pro por placa (cobre-borde 0,2 mm, alivios térmicos como aviso)
- fabricacion/*_gerber.zip: Gerbers + taladros PTH/NPTH desde el .kicad_pcb vigente; reemplazan los zips antiguos (los originales siguen en originales/)
- iBOM en español regenerado
- README y LEEME actualizados

Co-Authored-By: Claude Sonnet 5.5 <noreply@anthropic.com>
Claude-Session: https://claude.ai/code/session_01CUq9b9AsuT1a2cpCUYrCH3
Other:
- rule pad_to_mask_clearance: 0.051 -> 0
Changed lines of the file:
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@@
 		(rev "2")
 		(company "JJaroll.dev")
+		(comment 1 "Original: qbancoffee (LGPL-3.0) - Traduccion y firma: JJaroll.dev")
 		(comment 2 "audifonos, microfono, boton de encendido y 24 VAC")
 		(comment 3 "La placa J22 es una placa de conexiones para altavoces,")
 		(comment 4 "JJaroll.dev")
-		(comment 1 "Original: qbancoffee (LGPL-3.0) - Traduccion y firma: JJaroll.dev")
 	)
 	(layers
@@
 	)
 	(setup
-		(pad_to_mask_clearance 0.051)
-		(solder_mask_min_width 0.25)
+		(pad_to_mask_clearance 0)
 		(allow_soldermask_bridges_in_footprints no)
 		(tenting
@@
 			(disableapertmacros no)
 			(usegerberextensions no)
-			(usegerberattributes no)
+			(usegerberattributes yes)
 			(usegerberadvancedattributes no)
 			(creategerberjobfile no)

Commit message: Placas individuales: expansión de máscara 0,051 mm (como el diseño original)
- pad_to_mask_clearance 0,051 en los tres .kicad_pcb
- Gerbers de máscara ajustados con utilidades/expandir_mascara.py y verificados contra los Gerbers originales (diferencia de área de ~19 mm² a ~1,7 mm² por capa)
- LEEME de fabricacion y utilidades actualizados

Co-Authored-By: Claude Sonnet 5.5 <noreply@anthropic.com>
Claude-Session: https://claude.ai/code/session_01CUq9b9AsuT1a2cpCUYrCH3
Other:
- rule pad_to_mask_clearance: 0 -> 0.051
Changed lines of the file:
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@@
 	)
 	(setup
-		(pad_to_mask_clearance 0)
+		(pad_to_mask_clearance 0.051)
 		(allow_soldermask_bridges_in_footprints no)
 		(tenting
